File: desk_light/layout/LED_Lampe_v01.brd (EAGLE design)
At the start: 75 x 34 mm, 28 parts, among them IC1 LM1117DTX-ADJ, Q2 IRLML 2502

Commit message: changes to first prototype
Parts:
- added JP4: (no value), pinhead-1:1X02
- added JP5: (no value), pinhead-1:1X03
- added R12: 100R, resistor:R0805
- added TP1, TP10, TP2, TP3, TP4, TP5, TP6, TP7, TP8, TP9: TP-040, keystone:TP-040
- added U$2: PCA9530, i2c:SO08
- moved C1 19.3 mm to (5.46, 8.89)
- moved R11 19.2 mm to (33.0, 3.81), turned to 90 degrees
- moved R1 18.9 mm to (23.6, 12.6)
- moved R6 18.0 mm to (27.8, 6.99)
- moved D1 17.8 mm to (33.0, 8.89)
- moved R3 17.8 mm to (6.86, 3.43)
- moved R5 17.8 mm to (10.2, 3.43)
- moved R4 17.8 mm to (3.56, 3.43)
- moved U$1 17.8 mm to (16.5, 6.35)
- moved R2 17.3 mm to (19.6, 13.5), turned to 0 degrees
- moved L1 17.0 mm to (45.8, 7.49)
- moved C4 16.9 mm to (19.9, 2.54), turned to 180 degrees
- moved C3 16.8 mm to (11.3, 10.3)
- moved C2 16.6 mm to (24.8, 8.26), turned to 270 degrees
- moved Q2 16.2 mm to (24.5, 4.45), turned to 90 degrees
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Connections:
- removed net VDD: C5.+, D2.C, IC1.TAB, JP3.4, R7.2
- new net BLAAA: C5.+, D2.C, IC1.TAB, JP3.3, R12.1, R7.2, TP1.1, U$2.8
- new net DABLE: JP4.2, Q2.1, R11.1, TP6.1
- new net EXT: JP5.3
- new net N$10: R12.2, U$2.5
- new net N$11: JP3.1, U$2.7
- new net PWM0: JP5.1, U$2.2
- new net SCL: JP3.2, U$2.6
- net DIM: now also JP5.2, TP5.1; no longer JP3.2
- net DISABLE: now also JP4.1, U$2.3; no longer JP3.1, Q2.1, R11.1
- net GND: now also JP3.4, TP3.1, TP7.1, TP9.1, U$2.1, U$2.4; no longer JP3.3
- net N$6: now also TP4.1
- net N$9: now also TP10.1
- net VCC: now also TP2.1, TP8.1
Routing:
- net BLAAA: track 0.00 -> 68.7 mm, vias 0 -> 2
- net GND: track 117.2 -> 174.6 mm, vias 0 -> 2
- net N$9: track 18.1 -> 63.4 mm
- net N$6: track 0.00 -> 41.9 mm
- net N$8: track 3.92 -> 43.2 mm, vias 0 -> 2
- net DIM: track 0.00 -> 36.0 mm, vias 0 -> 2
- net VCC: track 59.1 -> 88.7 mm
- net N$11: track 0.00 -> 21.3 mm
- net VDD: track 21.0 -> 0.00 mm
- net N$62: track 0.00 -> 20.3 mm, vias 0 -> 2
- net N$54: track 0.00 -> 20.3 mm, vias 0 -> 3
- net SCL: track 0.00 -> 19.7 mm
- net DABLE: track 0.00 -> 18.6 mm
- net N$74: track 0.00 -> 17.8 mm
- net N$46: track 0.00 -> 17.8 mm, vias 0 -> 1
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- added copper zone on layer 1, net GND
- added copper zone on layer 1, net N$4
Other:
- board text added: "2012"
- board text added: "Mai"
- board text added: "v1.0"
