File: desk_light/layout/LED_Lampe_v01.sch (EAGLE design)
At the start: 28 parts, among them IC1 LM1117DTX-ADJ, Q2 IRLML 2502

Commit message: changes to first prototype
Parts:
- added JP4: (no value), pinhead-1:PINHD-1X2_2.54
- added JP5: (no value), pinhead-1:PINHD-1X3_2.54
- added R12: 100R, resistor:R-EU_R0805
- added TP1, TP10, TP2, TP3, TP4, TP5, TP6, TP7, TP8, TP9: TP-040, keystone:TP-040
- added U$2: PCA9530, i2c:PCA9530
Connections:
- removed net VDD: C5.+, D2.C, IC1.OUT, JP3.4, R7.2
- new net BLAAA: C5.+, D2.C, IC1.OUT, JP3.3, R12.1, R7.2, TP1.1, U$2.VCC
- new net DABLE: JP4.2, Q2.G, R11.1, TP6.1
- new net EXT: JP5.3
- new net N$10: R12.2, U$2.!RESET
- new net N$11: JP3.1, U$2.SDA
- new net PWM0: JP5.1, U$2.PWM0
- new net SCL: JP3.2, U$2.SCL
- net DIM: now also JP5.2, TP5.1; no longer JP3.2
- net DISABLE: now also JP4.1, U$2.PWM1; no longer JP3.1, Q2.G, R11.1
- net GND: now also JP3.4, TP3.1, TP7.1, TP9.1, U$2.A0, U$2.GND; no longer JP3.3
- net N$6: now also TP4.1
- net N$9: now also TP10.1
- net VCC: now also TP2.1, TP8.1
Other:
- note removed: "GND"
- note removed: "Vin"
- moved on the sheet: C5, C6, C7, D2, IC1, JP3, R10, R11, R7, R8, R9
