File: i2c_led_pcb_ng/LED.sch (EAGLE design)
At the start: 47 parts

Commit message: moved connector; bigger LED-pads for cooling; smaller address selector
Connections:
- net +3V3: no longer ADDR_SEL1.VCC, ADDR_SEL1.VCC@1, ADDR_SEL1.VCC@2
- net N$1: now also R1.1; no longer U$1RED.KATHODE
- net N$10: now also R10.1; no longer U$4RED.KATHODE
- net N$11: now also R11.1; no longer U$4GREEN.KATHODE
- net N$12: now also R12.1; no longer U$4BLUE.KATHODE
- net N$13: now also R12.2, U$4BLUE.KATHODE; no longer R3.1, U$1BLUE.ANODE
- net N$14: now also R11.2, U$4GREEN.KATHODE; no longer R2.1, U$1GREEN.ANODE
- net N$15: now also R10.2, U$4RED.KATHODE; no longer R1.1, U$1RED.ANODE
- net N$17: now also R7.2, U$3RED.KATHODE; no longer R6.1, U$2BLUE.ANODE
- net N$18: now also R8.2, U$3GREEN.KATHODE; no longer R5.1, U$2GREEN.ANODE
- net N$19: now also R2.2, U$1GREEN.KATHODE; no longer R4.1, U$2RED.ANODE
- net N$2: now also R2.1; no longer U$1GREEN.KATHODE
- net N$20: now also R1.2, U$1RED.KATHODE; no longer R9.1, U$3BLUE.ANODE
- net N$21: now also R3.2, U$1BLUE.KATHODE; no longer R8.1, U$3GREEN.ANODE
- net N$22: now also R4.2, U$2RED.KATHODE; no longer R7.1, U$3RED.ANODE
- net N$23: now also R5.2, U$2GREEN.KATHODE; no longer R12.1, U$4BLUE.ANODE
- net N$24: now also R6.2, U$2BLUE.KATHODE; no longer R11.1, U$4GREEN.ANODE
- net N$25: now also R13.2, U$11RED.KATHODE; no longer R10.1, U$4RED.ANODE
- net N$26: now also R13.1; no longer U$11RED.KATHODE
- net N$27: now also R14.1; no longer U$11GREEN.KATHODE
- net N$28: now also R15.1; no longer U$11BLUE.KATHODE
- net N$29: now also R16.1; no longer U$12RED.KATHODE
- net N$3: now also R3.1; no longer U$1BLUE.KATHODE
- net N$30: now also R17.1; no longer U$12GREEN.KATHODE
- net N$31: now also R18.1; no longer U$12BLUE.KATHODE
- net N$32: now also R19.1; no longer U$13RED.KATHODE
- net N$33: now also R20.1; no longer U$13GREEN.KATHODE
- net N$34: now also R21.1; no longer U$13BLUE.KATHODE
- net N$35: now also R22.1; no longer U$14RED.KATHODE
- net N$36: now also R23.1; no longer U$14GREEN.KATHODE
- net N$37: now also R24.1; no longer U$14BLUE.KATHODE
- net N$38: now also R14.2, U$11GREEN.KATHODE; no longer R15.1, U$11BLUE.ANODE
- net N$39: now also R15.2, U$11BLUE.KATHODE; no longer R14.1, U$11GREEN.ANODE
- net N$4: now also R4.1; no longer U$2RED.KATHODE
- net N$40: now also R16.2, U$12RED.KATHODE; no longer R13.1, U$11RED.ANODE
- net N$41: now also R17.2, U$12GREEN.KATHODE; no longer R18.1, U$12BLUE.ANODE
- net N$42: now also R18.2, U$12BLUE.KATHODE; no longer R17.1, U$12GREEN.ANODE
- net N$43: now also R24.2, U$14BLUE.KATHODE; no longer R16.1, U$12RED.ANODE
- net N$44: now also R23.2, U$14GREEN.KATHODE; no longer R21.1, U$13BLUE.ANODE
- net N$45: now also R22.2, U$14RED.KATHODE; no longer R20.1, U$13GREEN.ANODE
- net N$46: now also R21.2, U$13BLUE.KATHODE; no longer R19.1, U$13RED.ANODE
- net N$47: now also R20.2, U$13GREEN.KATHODE; no longer R24.1, U$14BLUE.ANODE
- net N$48: now also R19.2, U$13RED.KATHODE; no longer R23.1, U$14GREEN.ANODE
- net N$49: now also R9.2, U$3BLUE.KATHODE; no longer R22.1, U$14RED.ANODE
- net N$5: now also R5.1; no longer U$2GREEN.KATHODE
- net N$6: now also R6.1; no longer U$2BLUE.KATHODE
- net N$7: now also R7.1; no longer U$3RED.KATHODE
- net N$8: now also R8.1; no longer U$3GREEN.KATHODE
- net N$9: now also R9.1; no longer U$3BLUE.KATHODE
- net VCC: now also ADDR_SEL1.VCC, ADDR_SEL1.VCC@1, ADDR_SEL1.VCC@2, U$11BLUE.ANODE, U$11GREEN.ANODE, U$11RED.ANODE, U$12BLUE.ANODE, U$12GREEN.ANODE, U$12RED.ANODE, U$13BLUE.ANODE, U$13GREEN.ANODE, U$13RED.ANODE, U$14BLUE.ANODE, U$14GREEN.ANODE, U$14RED.ANODE, U$1BLUE.ANODE, U$1GREEN.ANODE, U$1RED.ANODE, U$2BLUE.ANODE, U$2GREEN.ANODE, U$2RED.ANODE, U$3BLUE.ANODE, U$3GREEN.ANODE, U$3RED.ANODE, U$4BLUE.ANODE, U$4GREEN.ANODE, U$4RED.ANODE; no longer R1.2, R10.2, R11.2, R12.2, R13.2, R14.2, R15.2, R16.2, R17.2, R18.2, R19.2, R2.2, R20.2, R21.2, R22.2, R23.2, R24.2, R3.2, R4.2, R5.2, R6.2, R7.2, R8.2, R9.2
Other:
- moved on the sheet: R1, R10, R11, R12, R13, R14, R15, R16, R17, R18, R19, R2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
